Commit message: Description with end effector

File: src/chipsy_description/urdf/chipsy_arm_body.xacro (robot description, xacro)
@@ -34,4 +34,9 @@
   <xacro:property name="wrist_roll_dia" value="0.1"/>
   <xacro:property name="wrist_roll_mass" value="0.1"/>
+  <!-- END EFFECTOR -->
+  <!-- along z axis -->
+  <xacro:property name="eef_length" value="0.1"/>
+  <xacro:property name="eef_width" value="0.025"/>
+  <xacro:property name="eef_mass" value="0.025"/>
   <xacro:property name="PI" value="3.141592653589793238"/>
   <!--///////////////////////////////////////////////////////////////////////-->
@@ -179,3 +184,53 @@
     <child link="wrist_roll_link"/>
   </joint>
+  <!--///////////////////////////////////////////////////////////////////////-->
+  <!-- RIGHT END EFFECTOR -->
+  <link name="right_eef_link">
+    <visual>
+      <origin xyz="0 0 ${eef_length/2}" rpy="0 0 0"/>
+      <geometry>
+        <box size="${eef_width} ${eef_width} ${eef_length}"/>
+      </geometry>
+      <material name="green"/>
+    </visual>
+    <collision>
+      <origin xyz="0 0 ${eef_length/2}" rpy="0 0 0"/>
+      <geometry>
+        <box size="${eef_width} ${eef_width} ${eef_length}"/>
+      </geometry>
+    </collision>
+    <xacro:base_inertial mass="${eef_mass}"/>
+  </link>
+  <joint name="right_eef_link_to_wrist_roll_link" type="prismatic">
+    <origin xyz="0 ${wrist_roll_dia/2} ${wrist_roll_length}" rpy="0 0 0"/>
+    <limit upper="${wrist_roll_dia/2-eef_width/2}" lower="${-wrist_roll_dia/2+eef_width/2}" effort="50" velocity="0.05"/>
+    <axis xyz="0 1 0" rpy="0 0 0"/>
+    <parent link="wrist_roll_link"/>
+    <child link="right_eef_link"/>
+  </joint>
+  <!--///////////////////////////////////////////////////////////////////////-->
+  <!-- LEFT END EFFECTOR -->
+  <link name="left_eef_link">
+    <visual>
+      <origin xyz="0 0 ${eef_length/2}" rpy="0 0 0"/>
+      <geometry>
+        <box size="${eef_width} ${eef_width} ${eef_length}"/>
+      </geometry>
+      <material name="green"/>
+    </visual>
+    <collision>
+      <origin xyz="0 0 ${eef_length/2}" rpy="0 0 0"/>
+      <geometry>
+        <box size="${eef_width} ${eef_width} ${eef_length}"/>
+      </geometry>
+    </collision>
+    <xacro:base_inertial mass="${eef_mass}"/>
+  </link>
+  <joint name="left_eef_link_to_wrist_roll_link" type="prismatic">
+    <origin xyz="0 ${-wrist_roll_dia/2} ${wrist_roll_length}" rpy="0 0 0"/>
+    <limit upper="${wrist_roll_dia/2-eef_width/2}" lower="${-wrist_roll_dia/2+eef_width/2}" effort="50" velocity="0.05"/>
+    <axis xyz="0 1 0" rpy="0 0 0"/>
+    <parent link="wrist_roll_link"/>
+    <child link="left_eef_link"/>
+  </joint>
 </robot>

Commit message: Add ros control to all joints

File: src/chipsy_description/urdf/chipsy_arm_body.xacro (robot description, xacro)
@@ -53,8 +53,10 @@
   <!--///////////////////////////////////////////////////////////////////////-->
   <!-- INERTIAL MACRO FOR ALL COMPONENTS -->
-  <xacro:macro name="base_inertial" params="mass">
+  <xacro:macro name="base_inertial" params="mass distance">
       <inertial>
+        <origin xyz="0 0 ${distance}" rpy="0 0 0"/>
       	<mass value="${mass}" />
-        <inertia ixx="1.0" ixy="0.0" ixz="0.0" iyy="0.5" iyz="0.0" izz="1.0" />
+        <!-- <inertia ixx="1.0" ixy="0.0" ixz="0.0" iyy="0.5" iyz="0.0" izz="1.0" /> -->
+        <inertia ixx="${0.1*mass}" ixy="0.0" ixz="0.0" iyy="${0.05*mass}" iyz="0.0" izz="${0.1*mass}" />
       </inertial>
    </xacro:macro>
@@ -78,7 +80,7 @@
       </geometry>
     </collision>
-    <xacro:base_inertial mass="${base_mass}"/>
-  </link>
-  <joint name="base_link_to_root_link" type="fixed">
+    <xacro:base_inertial mass="${base_mass}" distance="${base_height/2}"/>
+  </link>
+  <joint name="base_to_root_joint" type="fixed">
     <parent link="root_link"/>
     <child link="base_link"/>
@@ -100,7 +102,7 @@
       </geometry>
     </collision>
-    <xacro:base_inertial mass="${column_mass}"/>
-  </link>
-  <joint name="column_link_to_base_link" type="revolute">
+    <xacro:base_inertial mass="${column_mass}" distance="${column_length/2}"/>
+  </link>
+  <joint name="column_to_base_joint" type="revolute">
     <origin xyz="0 0 ${base_height}" rpy="0 0 0"/>
     <limit upper="${PI}" lower="${-1*PI}" effort="40" velocity="1"/>
@@ -109,4 +111,11 @@
     <child link="column_link"/>
   </joint>
+  <transmission name="column_to_base_transmission">
+    <type>transmission_interface/SimpleTransmission</type>
+    <joint name="column_to_base_joint">
+      <hardwareInterface>hardware_interface/EffortJointInterface</hardwareInterface>
+    </joint>
+    <actuator name="column_to_base_actuator"/>
+  </transmission>
   <!--///////////////////////////////////////////////////////////////////////-->
   <!-- UPPER ARM LINK -->
@@ -125,7 +134,7 @@
       </geometry>
     </collision>
-    <xacro:base_inertial mass="${upper_arm_mass}"/>
-  </link>
-  <joint name="upper_arm_link_to_column_link" type="revolute">
+    <xacro:base_inertial mass="${upper_arm_mass}" distance="${upper_arm_length/2}"/>
+  </link>
+  <joint name="upper_arm_to_column_joint" type="revolute">
     <origin xyz="0 0 ${column_length}" rpy="0 0 0"/>
     <limit upper="${PI}" lower="0" effort="20" velocity="1"/>
@@ -134,4 +143,11 @@
     <child link="upper_arm_link"/>
   </joint>
+  <transmission name="upper_arm_to_column_transmission">
+    <type>transmission_interface/SimpleTransmission</type>
+    <joint name="upper_arm_to_column_joint">
+      <hardwareInterface>hardware_interface/EffortJointInterface</hardwareInterface>
+    </joint>
+    <actuator name="upper_arm_to_column_actuator"/>
+  </transmission>
   <!--///////////////////////////////////////////////////////////////////////-->
   <!-- LOWER ARM LINK -->
@@ -150,7 +166,7 @@
       </geometry>
     </collision>
-    <xacro:base_inertial mass="${lower_arm_mass}"/>
-  </link>
-  <joint name="lower_arm_link_to_upper_arm_link" type="revolute">
+    <xacro:base_inertial mass="${lower_arm_mass}" distance="${lower_arm_length/2}"/>
+  </link>
+  <joint name="lower_arm_to_upper_arm_joint" type="revolute">
     <origin xyz="0 0 ${upper_arm_length}" rpy="0 0 0"/>
     <limit upper="${PI}" lower="0" effort="20" velocity="1"/>
@@ -159,4 +175,11 @@
     <child link="lower_arm_link"/>
   </joint>
+  <transmission name="lower_arm_to_upper_arm_transmission">
+    <type>transmission_interface/SimpleTransmission</type>
+    <joint name="lower_arm_to_upper_arm_joint">
+      <hardwareInterface>hardware_interface/EffortJointInterface</hardwareInterface>
+    </joint>
+    <actuator name="lower_arm_to_upper_arm_actuator"/>
+  </transmission>
   <!--///////////////////////////////////////////////////////////////////////-->
   <!-- WRIST ROLL LINK -->
@@ -175,7 +198,7 @@
       </geometry>
     </collision>
-    <xacro:base_inertial mass="${wrist_roll_mass}"/>
-  </link>
-  <joint name="wrist_roll_link_to_upper_arm_link" type="revolute">
+    <xacro:base_inertial mass="${wrist_roll_mass}" distance="${wrist_roll_length/2}"/>
+  </link>
+  <joint name="wrist_roll_to_lower_arm_joint" type="revolute">
     <origin xyz="0 0 ${lower_arm_length}" rpy="0 0 0"/>
     <limit upper="${PI}" lower="${-1*PI}" effort="20" velocity="1"/>
@@ -184,4 +207,14 @@
     <child link="wrist_roll_link"/>
   </joint>
+  <transmission name="wrist_roll_to_lower_arm_transmission">
+    <type>transmission_interface/SimpleTransmission</type>
+    <joint name="wrist_roll_to_lower_arm_joint">
+      <hardwareInterface>hardware_interface/EffortJointInterface</hardwareInterface>
+    </joint>
+    <actuator name="wrist_roll_to_lower_arm_actuator"/>
+  </transmission>
+  <gazebo reference="wrist_roll_link">
+    <material>Gazebo/Red</material>
+  </gazebo>
   <!--///////////////////////////////////////////////////////////////////////-->
   <!-- RIGHT END EFFECTOR -->
@@ -200,7 +233,7 @@
       </geometry>
     </collision>
-    <xacro:base_inertial mass="${eef_mass}"/>
-  </link>
-  <joint name="right_eef_link_to_wrist_roll_link" type="prismatic">
+    <xacro:base_inertial mass="${eef_mass}" distance="${eef_length/2}"/>
+  </link>
+  <joint name="right_eef_to_wrist_roll_joint" type="prismatic">
     <origin xyz="0 ${wrist_roll_dia/2} ${wrist_roll_length}" rpy="0 0 0"/>
     <limit upper="${wrist_roll_dia/2-eef_width/2}" lower="${-wrist_roll_dia/2+eef_width/2}" effort="50" velocity="0.05"/>
@@ -209,4 +242,11 @@
     <child link="right_eef_link"/>
   </joint>
+  <transmission name="right_eef_to_wrist_roll_transmission">
+    <type>transmission_interface/SimpleTransmission</type>
+    <joint name="right_eef_to_wrist_roll_joint">
+      <hardwareInterface>hardware_interface/EffortJointInterface</hardwareInterface>
+    </joint>
+    <actuator name="right_eef_to_wrist_roll_actuator"/>
+  </transmission>
   <!--///////////////////////////////////////////////////////////////////////-->
   <!-- LEFT END EFFECTOR -->
@@ -225,7 +265,7 @@
       </geometry>
     </collision>
-    <xacro:base_inertial mass="${eef_mass}"/>
-  </link>
-  <joint name="left_eef_link_to_wrist_roll_link" type="prismatic">
+    <xacro:base_inertial mass="${eef_mass}" distance="${eef_length/2}"/>
+  </link>
+  <joint name="left_eef_to_wrist_roll_joint" type="prismatic">
     <origin xyz="0 ${-wrist_roll_dia/2} ${wrist_roll_length}" rpy="0 0 0"/>
     <limit upper="${wrist_roll_dia/2-eef_width/2}" lower="${-wrist_roll_dia/2+eef_width/2}" effort="50" velocity="0.05"/>
@@ -234,3 +274,15 @@
     <child link="left_eef_link"/>
   </joint>
+  <transmission name="left_eef_to_wrist_roll_transmission">
+    <type>transmission_interface/SimpleTransmission</type>
+    <joint name="left_eef_to_wrist_roll_joint">
+      <hardwareInterface>hardware_interface/EffortJointInterface</hardwareInterface>
+    </joint>
+    <actuator name="left_eef_to_wrist_roll_actuator"/>
+  </transmission>
+  <!--///////////////////////////////////////////////////////////////////////-->
+  <!-- ROS CONTROL PLUGIN -->
+  <gazebo>
+    <plugin name="gazebo_ros_control" filename="libgazebo_ros_control.so"/>
+  </gazebo>
 </robot>

Commit message: Multi model spawning

File: src/chipsy_description/urdf/chipsy_arm_body.xacro (robot description, xacro)
@@ -1,7 +1,4 @@
 <?xml version="1.0"?>
-<robot name="chipsy_arm" xmlns:xacro="http://ros.org/wiki/xacro"
-            xmlns:sensor="http://playerstage.sourceforge.net/gazebo/xmlschema/#sensor"
-            xmlns:controller="http://playerstage.sourceforge.net/gazebo/xmlschema/#controller"
-            xmlns:interface="http://playerstage.sourceforge.net/gazebo/xmlschema/#interface">
+<robot name="chipsy_arm" xmlns:xacro="http://ros.org/wiki/xacro">
   <!--///////////////////////////////////////////////////////////////////////-->
   <!-- GENERIC PROPERTIES USED IN THE ARM -->
@@ -64,4 +61,10 @@
   <!-- DUMMY ROOT LINK SO THAT BASE LINK CAN BE GIVEN SOME MASS -->
   <link name="root_link"/>
+  <!-- FIXING ROBOT TO THE WORLD' -->
+  <link name="world"/>
+  <joint name="fixed" type="fixed">
+    <parent link="world"/>
+    <child link="root_link"/>
+  </joint>
   <!--///////////////////////////////////////////////////////////////////////-->
   <!-- BASE LINK IS THE LINK WHICH EVERYTHING IS ATTACHED TO -->
@@ -286,3 +289,11 @@
     <plugin name="gazebo_ros_control" filename="libgazebo_ros_control.so"/>
   </gazebo>
+  <!-- JOINT STATE PUBLISHER -->
+  <gazebo>
+    <plugin name="joint_state_publisher" filename="libgazebo_ros_joint_state_publisher.so">
+      <jointName>column_to_base_joint,upper_arm_to_column_joint,
+      lower_arm_to_upper_arm_joint, wrist_roll_to_lower_arm_joint,
+      right_eef_to_wrist_roll_joint, left_eef_to_wrist_roll_joint</jointName>
+    </plugin>
+  </gazebo>
 </robot>
