Commit message: Complete conveyor belt

File: src/chipsy_description/urdf/chipsy_conveyor.xacro (robot description, xacro)
@@ -5,5 +5,5 @@
   <xacro:property name="base_length" value="0.5"/>
   <!-- along y axis -->
-  <xacro:property name="base_width" value="0.5"/>
+  <xacro:property name="base_width" value="5"/>
   <!-- along z axis -->
   <xacro:property name="base_height" value="0.1"/>
@@ -12,8 +12,10 @@
   <xacro:property name="belt_length" value="0.5"/>
   <!-- along y axis -->
-  <xacro:property name="belt_width" value="0.5"/>
+  <xacro:property name="belt_width" value="5"/>
   <!-- along z axis -->
-  <xacro:property name="belt_height" value="0.05"/>
+  <xacro:property name="belt_height" value="0.005"/>
   <xacro:property name="belt_mass" value="2.5"/>
+  <!-- Set the limit of the belt and base joint -->
+  <xacro:property name="belt_limit" value="5"/>
   <xacro:property name="PI" value="3.141592653589793238"/>
   <!-- COLOURS FOR MATERIAL -->
@@ -77,5 +79,5 @@
   <link name="belt_link">
     <visual>
-      <origin xyz="0 0 ${belt_height/2}" rpy="0 0 0"/>
+      <origin xyz="0 ${-base_width/2} ${belt_height/2}" rpy="0 0 0"/>
       <geometry>
         <box size="${belt_length} ${belt_width} ${belt_height}"/>
@@ -84,5 +86,5 @@
     </visual>
     <collision>
-      <origin xyz="0 0 ${belt_height/2}" rpy="0 0 0"/>
+      <origin xyz="0 ${-base_width/2} ${belt_height/2}" rpy="0 0 0"/>
       <geometry>
         <box size="${belt_length} ${belt_width} ${belt_height}"/>
@@ -94,5 +96,5 @@
   <joint name="belt_to_base_joint" type="prismatic">
     <origin xyz="0 0 ${base_height}" rpy="0 0 0"/>
-    <limit upper="${PI}" lower="${-1*PI}" effort="20" velocity="1"/>
+    <limit upper="${belt_limit}" lower="${-1*belt_limit}" effort="20" velocity="1"/>
     <axis xyz="0 1 0" rpy="0 0 0"/>
     <parent link="base_link"/>
@@ -104,9 +106,9 @@
   </gazebo>
   <!-- TESTING THE CUSTOM CONVEYOR BELT PLUGIN -->
-  <!-- <gazebo>
+  <gazebo>
     <plugin name="ConveyorBeltPlugin" filename="/home/raghav/chipsy/devel/lib/libConveyorBeltPlugin.so">
     <belt_joint>belt_to_base_joint</belt_joint>
   </plugin>
-  </gazebo> -->
+  </gazebo>
   <!-- JOINT STATE PUBLISHER -->
   <gazebo>

File: src/chipsy_description/urdf/chipsy_ugv.xacro (robot description, xacro)
@@ -100,4 +100,21 @@
   </plugin>
   </gazebo> -->
+  <!-- SKID STEER PLUGIN -->
+  <gazebo>
+    <plugin name="skid_steer_drive_controller" filename="libgazebo_ros_skid_steer_drive.so">
+      <updateRate>100.0</updateRate>
+      <robotNamespace>/chipsy_ugv</robotNamespace>
+      <leftFrontJoint>left_front_wheel_to_base_link</leftFrontJoint>
+      <rightFrontJoint>right_front_wheel_to_base_link</rightFrontJoint>
+      <leftRearJoint>left_back_wheel_to_base_link</leftRearJoint>
+      <rightRearJoint>right_back_wheel_to_base_link</rightRearJoint>
+      <wheelSeparation>0.5</wheelSeparation>
+      <wheelDiameter>0.1</wheelDiameter>
+      <robotBaseFrame>base_link</robotBaseFrame>
+      <torque>5</torque>
+      <commandTopic>cmd_vel</commandTopic>
+      <broadcastTF>false</broadcastTF>
+    </plugin>
+  </gazebo>
   <!-- JOINT STATE PUBLISHER -->
   <gazebo>
