Commit message: cleanup

File: src/chipsy_description/urdf/chipsy_ugv.xacro (robot description, xacro)
@@ -76,5 +76,5 @@
       <material name="white"/>
     </visual>
-    <collision>
+    <collision name="base_link_collision">
       <origin xyz="0 0 ${wheel_dia + base_height/2}" rpy="0 0 0"/>
       <geometry>
@@ -117,4 +117,16 @@
     </plugin>
   </gazebo>
+  <!-- <gazebo reference="base_link">
+    <sensor type="contact" name="ContactPlugin">
+      <selfCollide>true</selfCollide>
+      <alwaysOn>true</alwaysOn>
+      <updateRate>15.0</updateRate>
+      <material>Gazebo/Red</material>
+      <contact>
+       <collision>base_link_collision</collision>
+      </contact>
+      <plugin name="ContactPlugin" filename="libContactPlugin.so"/>
+    </sensor>
+  </gazebo> -->
   <!-- JOINT STATE PUBLISHER -->
   <gazebo>
