Commit message: add details to param server, start ik

File: src/chipsy_description/urdf/chipsy_arm.xacro (robot description, xacro)
@@ -109,5 +109,5 @@
   <joint name="column_to_base_joint" type="revolute">
     <origin xyz="0 0 ${base_height}" rpy="0 0 0"/>
-    <limit upper="${PI}" lower="${-1*PI}" effort="40" velocity="1"/>
+    <limit upper="${PI}" lower="${-1*PI}" effort="400" velocity="10"/>
     <axis xyz="0 0 1" rpy="0 0 0"/>
     <parent link="base_link"/>

Commit message: Rudimentary IK

File: src/chipsy_description/urdf/chipsy_arm.xacro (robot description, xacro)
@@ -18,10 +18,10 @@
   <!-- UPPER ARM -->
   <!-- along z axis -->
-  <xacro:property name="upper_arm_length" value="0.25"/>
+  <xacro:property name="upper_arm_length" value="0.4"/>
   <xacro:property name="upper_arm_dia" value="0.1"/>
   <xacro:property name="upper_arm_mass" value="0.5"/>
   <!-- LOWER ARM -->
   <!-- along z axis -->
-  <xacro:property name="lower_arm_length" value="0.25"/>
+  <xacro:property name="lower_arm_length" value="0.4"/>
   <xacro:property name="lower_arm_dia" value="0.1"/>
   <xacro:property name="lower_arm_mass" value="0.5"/>
@@ -141,5 +141,5 @@
   <joint name="upper_arm_to_column_joint" type="revolute">
     <origin xyz="0 0 ${column_length}" rpy="0 0 0"/>
-    <limit upper="${PI}" lower="0" effort="20" velocity="1"/>
+    <limit upper="${PI}" lower="0" effort="100" velocity="1"/>
     <axis xyz="0 1 0" rpy="0 0 0"/>
     <parent link="column_link"/>
@@ -173,5 +173,5 @@
   <joint name="lower_arm_to_upper_arm_joint" type="revolute">
     <origin xyz="0 0 ${upper_arm_length}" rpy="0 0 0"/>
-    <limit upper="${PI}" lower="0" effort="20" velocity="1"/>
+    <limit upper="${PI}" lower="0" effort="100" velocity="1"/>
     <axis xyz="0 1 0" rpy="0 0 0"/>
     <parent link="upper_arm_link"/>

File: src/chipsy_description/urdf/chipsy_conveyor.xacro (robot description, xacro)
@@ -7,5 +7,5 @@
   <xacro:property name="base_width" value="5"/>
   <!-- along z axis -->
-  <xacro:property name="base_height" value="0.1"/>
+  <xacro:property name="base_height" value="0.25"/>
   <xacro:property name="base_mass" value="5"/>
   <!-- along x axis -->
